File: led-board/led-board.kicad_pcb (KiCad board)
At the start: 2 copper layers, 0 parts

Commit message: Layout complete
Parts:
- added C1: 0.1u, Capacitor_SMD:C_0603_1608Metric, F.Cu at (294.5, 198.5)
- added C10: 0.1u, Capacitor_SMD:C_0603_1608Metric, F.Cu at (220.0, 231.5)
- added C100: 470n, Capacitor_SMD:C_0603_1608Metric, F.Cu at (85.0, 136.6)
- added C101: 4.7n, Capacitor_SMD:C_0603_1608Metric, F.Cu at (85.0, 133.2)
- added C102: 0.1u, Capacitor_SMD:C_0603_1608Metric, F.Cu at (190.0, 141.5)
- added C103: 0.1u, Capacitor_SMD:C_0603_1608Metric, F.Cu at (190.0, 156.5)
- added C104: 0.1u, Capacitor_SMD:C_0603_1608Metric, F.Cu at (280.0, 141.5)
- added C105: 0.1u, Capacitor_SMD:C_0603_1608Metric, F.Cu at (280.0, 156.5)
- added C106: 0.1u, Capacitor_SMD:C_0603_1608Metric, F.Cu at (175.0, 141.5)
- added C107: 0.1u, Capacitor_SMD:C_0603_1608Metric, F.Cu at (175.0, 156.5)
- added C108: 0.1u, Capacitor_SMD:C_0603_1608Metric, F.Cu at (265.0, 141.5)
- added C109: 0.1u, Capacitor_SMD:C_0603_1608Metric, F.Cu at (265.0, 156.5)
- added C11: 10u, Capacitor_SMD:C_0603_1608Metric, F.Cu at (284.5, 222.5)
- added C110: 10u, Capacitor_SMD:C_0603_1608Metric, F.Cu at (95.8, 147.2)
- added C111: 10u, Capacitor_SMD:C_0603_1608Metric, F.Cu at (94.6, 131.3)
- added C112: 0.1u, Capacitor_SMD:C_0603_1608Metric, F.Cu at (160.0, 141.5)
- added C113: 0.1u, Capacitor_SMD:C_0603_1608Metric, F.Cu at (160.0, 156.5)
- added C114: 0.1u, Capacitor_SMD:C_0603_1608Metric, F.Cu at (250.0, 141.5)
- added C115: 0.1u, Capacitor_SMD:C_0603_1608Metric, F.Cu at (250.0, 156.5)
- added C116: 0.1u, Capacitor_SMD:C_0603_1608Metric, F.Cu at (92.2, 147.2)
- added C117: 0.1u, Capacitor_SMD:C_0603_1608Metric, F.Cu at (91.2, 131.3)
- added C118: 0.1u, Capacitor_SMD:C_0603_1608Metric, F.Cu at (145.0, 141.5)
- added C119: 0.1u, Capacitor_SMD:C_0603_1608Metric, F.Cu at (145.0, 156.5)
- added C12: 1u, Capacitor_SMD:C_0603_1608Metric, F.Cu at (278.5, 237.2)
- added C120: 0.1u, Capacitor_SMD:C_0603_1608Metric, F.Cu at (235.0, 141.5)
- added C121: 0.1u, Capacitor_SMD:C_0603_1608Metric, F.Cu at (235.0, 156.5)
- added C122: 0.1u, Capacitor_SMD:C_0603_1608Metric, F.Cu at (130.0, 141.5)
- added C123: 0.1u, Capacitor_SMD:C_0603_1608Metric, F.Cu at (130.0, 156.5)
- added C124: 0.1u, Capacitor_SMD:C_0603_1608Metric, F.Cu at (220.0, 141.5)
- added C125: 0.1u, Capacitor_SMD:C_0603_1608Metric, F.Cu at (220.0, 156.5)
- added C126: 0.1u, Capacitor_SMD:C_0603_1608Metric, F.Cu at (150.4, 73.2)
- added C127: 0.1u, Capacitor_SMD:C_0603_1608Metric, F.Cu at (118.2, 77.4)
- added C128: 0.1u, Capacitor_SMD:C_0603_1608Metric, F.Cu at (291.5, 214.2)
- added C129: 220u, Capacitor_SMD:CP_Elec_10x10, F.Cu at (136.7, 69.0)
- added C13: 1u, Capacitor_SMD:C_0603_1608Metric, F.Cu at (281.3, 237.2)
- added C130: 220u, Capacitor_SMD:CP_Elec_10x10, F.Cu at (134.5, 80.4)
- added C131: 220u, Capacitor_SMD:CP_Elec_10x10, F.Cu at (297.1, 56.5)
- added C132: 220u, Capacitor_SMD:CP_Elec_10x10, F.Cu at (285.9, 56.5)
- added C133: 0.1u, Capacitor_SMD:C_0603_1608Metric, F.Cu at (279.1, 52.5)
- added C134: 220u, Capacitor_SMD:CP_Elec_10x10, F.Cu at (276.9, 69.1)
- added C135: 220u, Capacitor_SMD:CP_Elec_10x10, F.Cu at (280.0, 84.2)
- added C136: 220u, Capacitor_SMD:CP_Elec_10x10, F.Cu at (268.4, 84.2)
- added C137: 0.1u, Capacitor_SMD:C_0603_1608Metric, F.Cu at (286.6, 88.0)
- added C138: 220u, Capacitor_SMD:CP_Elec_10x10, F.Cu at (288.6, 71.2)
- added C14: 0.1u, Capacitor_SMD:C_0603_1608Metric, F.Cu at (190.0, 81.5)
- added C15: 0.1u, Capacitor_SMD:C_0603_1608Metric, F.Cu at (205.0, 216.5)
- added C16: 0.1u, Capacitor_SMD:C_0603_1608Metric, F.Cu at (235.0, 81.5)
- added C17: 0.1u, Capacitor_SMD:C_0603_1608Metric, F.Cu at (235.0, 216.5)
- added C18: 0.1u, Capacitor_SMD:C_0603_1608Metric, F.Cu at (284.1, 237.2)
- added C19: 22u, Capacitor_SMD:C_0603_1608Metric, F.Cu at (280.5, 222.5)
- added C2: 0.1u, Capacitor_SMD:C_0603_1608Metric, F.Cu at (303.0, 180.7)
- added C20: 0.1u, Capacitor_SMD:C_0603_1608Metric, F.Cu at (205.0, 81.5)
- added C21: 0.1u, Capacitor_SMD:C_0603_1608Metric, F.Cu at (190.0, 216.5)
- added C22: 0.1u, Capacitor_SMD:C_0603_1608Metric, F.Cu at (220.0, 81.5)
- added C23: 0.1u, Capacitor_SMD:C_0603_1608Metric, F.Cu at (220.0, 216.5)
- added C24: 0.1u, Capacitor_SMD:C_0603_1608Metric, F.Cu at (205.0, 96.5)
- added C25: 0.1u, Capacitor_SMD:C_0603_1608Metric, F.Cu at (205.0, 201.5)
- added C26: 0.1u, Capacitor_SMD:C_0603_1608Metric, F.Cu at (250.0, 96.5)
- added C27: 0.1u, Capacitor_SMD:C_0603_1608Metric, F.Cu at (250.0, 201.5)
- added C28: 0.1u, Capacitor_SMD:C_0603_1608Metric, F.Cu at (190.0, 96.5)
- added C29: 0.1u, Capacitor_SMD:C_0603_1608Metric, F.Cu at (190.0, 201.5)
- added C3: 22p, Capacitor_SMD:C_0603_1608Metric, F.Cu at (282.5, 193.2)
- added C30: 0.1u, Capacitor_SMD:C_0603_1608Metric, F.Cu at (235.0, 96.5)
- added C31: 0.1u, Capacitor_SMD:C_0603_1608Metric, F.Cu at (235.0, 201.5)
- added C32: 0.1u, Capacitor_SMD:C_0603_1608Metric, F.Cu at (175.0, 96.5)
- added C33: 0.1u, Capacitor_SMD:C_0603_1608Metric, F.Cu at (175.0, 201.5)
- added C34: 0.1u, Capacitor_SMD:C_0603_1608Metric, F.Cu at (220.0, 96.5)
- added C35: 0.1u, Capacitor_SMD:C_0603_1608Metric, F.Cu at (220.0, 201.5)
- added C36: 0.1u, Capacitor_SMD:C_0603_1608Metric, F.Cu at (205.0, 111.5)
- added C37: 0.1u, Capacitor_SMD:C_0603_1608Metric, F.Cu at (205.0, 186.5)
- added C38: 0.1u, Capacitor_SMD:C_0603_1608Metric, F.Cu at (265.0, 111.5)
- added C39: 0.1u, Capacitor_SMD:C_0603_1608Metric, F.Cu at (265.0, 186.5)
- added C4: 22p, Capacitor_SMD:C_0603_1608Metric, F.Cu at (274.5, 193.2)
- added C40: 220u, Capacitor_SMD:CP_Elec_10x10, F.Cu at (150.4, 90.5)
- added C41: 0.1u, Capacitor_SMD:C_0603_1608Metric, F.Cu at (190.0, 111.5)
- added C42: 0.1u, Capacitor_SMD:C_0603_1608Metric, F.Cu at (190.0, 186.5)
- added C43: 0.1u, Capacitor_SMD:C_0603_1608Metric, F.Cu at (250.0, 111.5)
- added C44: 0.1u, Capacitor_SMD:C_0603_1608Metric, F.Cu at (250.0, 186.5)
- added C45: 0.1u, Capacitor_SMD:C_0603_1608Metric, F.Cu at (298.5, 214.2)
- added C46: 0.1u, Capacitor_SMD:C_0603_1608Metric, F.Cu at (284.0, 214.2)
- added C47: 0.1u, Capacitor_SMD:C_0603_1608Metric, F.Cu at (175.0, 111.5)
- added C48: 0.1u, Capacitor_SMD:C_0603_1608Metric, F.Cu at (175.0, 186.5)
- added C49: 0.1u, Capacitor_SMD:C_0603_1608Metric, F.Cu at (235.0, 111.5)
- added C5: 0.1u, Capacitor_SMD:C_0603_1608Metric, F.Cu at (286.2, 197.8)
- added C50: 0.1u, Capacitor_SMD:C_0603_1608Metric, F.Cu at (235.0, 186.5)
- added C51: 0.1u, Capacitor_SMD:C_0603_1608Metric, F.Cu at (343.2, 151.5)
- added C52: 0.1u, Capacitor_SMD:C_0603_1608Metric, F.Cu at (343.2, 135.0)
- added C53: 220u, Capacitor_SMD:CP_Elec_10x10, F.Cu at (122.4, 70.8)
- added C54: 0.1u, Capacitor_SMD:C_0603_1608Metric, F.Cu at (160.0, 111.5)
- added C55: 0.1u, Capacitor_SMD:C_0603_1608Metric, F.Cu at (160.0, 186.5)
- added C56: 0.1u, Capacitor_SMD:C_0603_1608Metric, F.Cu at (220.0, 111.5)
- added C57: 0.1u, Capacitor_SMD:C_0603_1608Metric, F.Cu at (220.0, 186.5)
- added C58: 220u, Capacitor_SMD:CP_Elec_10x10, F.Cu at (150.4, 79.5)
- added C59: 4.7n, Capacitor_SMD:C_0603_1608Metric, F.Cu at (339.5, 150.0)
- added C6: 0.1u, Capacitor_SMD:C_0603_1608Metric, F.Cu at (284.2, 197.8)
- added C60: 470n, Capacitor_SMD:C_0603_1608Metric, F.Cu at (339.5, 153.2)
- added C61: 4.7n, Capacitor_SMD:C_0603_1608Metric, F.Cu at (339.5, 156.5)
- added C62: 4.7n, Capacitor_SMD:C_0603_1608Metric, F.Cu at (339.2, 133.0)
- added C63: 470n, Capacitor_SMD:C_0603_1608Metric, F.Cu at (339.2, 136.5)
- added C64: 4.7n, Capacitor_SMD:C_0603_1608Metric, F.Cu at (339.2, 140.0)
- added C65: 0.1u, Capacitor_SMD:C_0603_1608Metric, F.Cu at (205.0, 126.5)
- added C66: 0.1u, Capacitor_SMD:C_0603_1608Metric, F.Cu at (205.0, 171.5)
- added C67: 0.1u, Capacitor_SMD:C_0603_1608Metric, F.Cu at (280.0, 126.5)
- added C68: 0.1u, Capacitor_SMD:C_0603_1608Metric, F.Cu at (280.0, 171.5)
- added C69: 0.1u, Capacitor_SMD:C_0603_1608Metric, F.Cu at (190.0, 126.5)
- added C7: 0.1u, Capacitor_SMD:C_0603_1608Metric, F.Cu at (205.0, 66.5)
- added C70: 0.1u, Capacitor_SMD:C_0603_1608Metric, F.Cu at (190.0, 171.5)
- added C71: 0.1u, Capacitor_SMD:C_0603_1608Metric, F.Cu at (265.0, 126.5)
- added C72: 0.1u, Capacitor_SMD:C_0603_1608Metric, F.Cu at (265.0, 171.5)
- added C73: 10u, Capacitor_SMD:C_0603_1608Metric, F.Cu at (330.2, 158.5)
- added C74: 10u, Capacitor_SMD:C_0603_1608Metric, F.Cu at (329.2, 142.0)
- added C75: 220u, Capacitor_SMD:CP_Elec_10x10, F.Cu at (122.4, 59.6)
- added C76: 0.1u, Capacitor_SMD:C_0603_1608Metric, F.Cu at (175.0, 126.5)
- added C77: 0.1u, Capacitor_SMD:C_0603_1608Metric, F.Cu at (175.0, 171.5)
- added C78: 0.1u, Capacitor_SMD:C_0603_1608Metric, F.Cu at (250.0, 126.5)
- added C79: 0.1u, Capacitor_SMD:C_0603_1608Metric, F.Cu at (250.0, 171.5)
- added C8: 0.1u, Capacitor_SMD:C_0603_1608Metric, F.Cu at (205.0, 231.5)
- added C80: 0.1u, Capacitor_SMD:C_0603_1608Metric, F.Cu at (333.5, 158.5)
- added C81: 0.1u, Capacitor_SMD:C_0603_1608Metric, F.Cu at (332.8, 142.0)
- added C82: 0.1u, Capacitor_SMD:C_0603_1608Metric, F.Cu at (160.0, 126.5)
- added C83: 0.1u, Capacitor_SMD:C_0603_1608Metric, F.Cu at (160.0, 171.5)
- added C84: 0.1u, Capacitor_SMD:C_0603_1608Metric, F.Cu at (235.0, 126.5)
- added C85: 0.1u, Capacitor_SMD:C_0603_1608Metric, F.Cu at (235.0, 171.5)
- added C86: 0.1u, Capacitor_SMD:C_0603_1608Metric, F.Cu at (145.0, 126.5)
- added C87: 0.1u, Capacitor_SMD:C_0603_1608Metric, F.Cu at (145.0, 171.5)
- added C88: 0.1u, Capacitor_SMD:C_0603_1608Metric, F.Cu at (220.0, 126.5)
- added C89: 0.1u, Capacitor_SMD:C_0603_1608Metric, F.Cu at (220.0, 171.5)
- added C9: 0.1u, Capacitor_SMD:C_0603_1608Metric, F.Cu at (220.0, 66.5)
- added C90: 0.1u, Capacitor_SMD:C_0603_1608Metric, F.Cu at (81.8, 154.8)
- added C91: 0.1u, Capacitor_SMD:C_0603_1608Metric, F.Cu at (81.2, 138.2)
- added C92: 0.1u, Capacitor_SMD:C_0603_1608Metric, F.Cu at (205.0, 141.5)
- added C93: 0.1u, Capacitor_SMD:C_0603_1608Metric, F.Cu at (205.0, 156.5)
- added C94: 0.1u, Capacitor_SMD:C_0603_1608Metric, F.Cu at (295.0, 141.5)
- added C95: 0.1u, Capacitor_SMD:C_0603_1608Metric, F.Cu at (295.0, 156.5)
- added C96: 4.7n, Capacitor_SMD:C_0603_1608Metric, F.Cu at (85.8, 156.8)
- added C97: 470n, Capacitor_SMD:C_0603_1608Metric, F.Cu at (85.8, 152.8)
- added C98: 4.7n, Capacitor_SMD:C_0603_1608Metric, F.Cu at (85.8, 149.2)
- added C99: 4.7n, Capacitor_SMD:C_0603_1608Metric, F.Cu at (85.0, 139.9)
- added D1: LED_Small, LED_SMD:LED_0603_1608Metric, F.Cu at (263.5, 205.8)
- added D10: WS2813, LED_SMD:LED_WS2812_PLCC6_5.0x5.0mm_P1.6mm, F.Cu at (235.0, 77.5)
- added D11: WS2813, LED_SMD:LED_WS2812_PLCC6_5.0x5.0mm_P1.6mm, F.Cu at (235.0, 212.5)
- added D12: WS2813, LED_SMD:LED_WS2812_PLCC6_5.0x5.0mm_P1.6mm, F.Cu at (190.0, 77.5)
- added D13: WS2813, LED_SMD:LED_WS2812_PLCC6_5.0x5.0mm_P1.6mm, F.Cu at (190.0, 212.5)
- added D14: WS2813, LED_SMD:LED_WS2812_PLCC6_5.0x5.0mm_P1.6mm, F.Cu at (220.0, 77.5)
- added D15: WS2813, LED_SMD:LED_WS2812_PLCC6_5.0x5.0mm_P1.6mm, F.Cu at (220.0, 212.5)
- added D16: WS2813, LED_SMD:LED_WS2812_PLCC6_5.0x5.0mm_P1.6mm, F.Cu at (205.0, 92.5)
- added D17: WS2813, LED_SMD:LED_WS2812_PLCC6_5.0x5.0mm_P1.6mm, F.Cu at (205.0, 197.5)
- added D18: WS2813, LED_SMD:LED_WS2812_PLCC6_5.0x5.0mm_P1.6mm, F.Cu at (250.0, 92.5)
- added D19: WS2813, LED_SMD:LED_WS2812_PLCC6_5.0x5.0mm_P1.6mm, F.Cu at (250.0, 197.5)
- added D2: LED_Small, LED_SMD:LED_0603_1608Metric, F.Cu at (263.5, 208.8)
- added D20: WS2813, LED_SMD:LED_WS2812_PLCC6_5.0x5.0mm_P1.6mm, F.Cu at (190.0, 92.5)
- added D21: WS2813, LED_SMD:LED_WS2812_PLCC6_5.0x5.0mm_P1.6mm, F.Cu at (190.0, 197.5)
- added D22: WS2813, LED_SMD:LED_WS2812_PLCC6_5.0x5.0mm_P1.6mm, F.Cu at (235.0, 92.5)
- added D23: WS2813, LED_SMD:LED_WS2812_PLCC6_5.0x5.0mm_P1.6mm, F.Cu at (235.0, 197.5)
- added D24: WS2813, LED_SMD:LED_WS2812_PLCC6_5.0x5.0mm_P1.6mm, F.Cu at (175.0, 92.5)
- added D25: WS2813, LED_SMD:LED_WS2812_PLCC6_5.0x5.0mm_P1.6mm, F.Cu at (175.0, 197.5)
- added D26: WS2813, LED_SMD:LED_WS2812_PLCC6_5.0x5.0mm_P1.6mm, F.Cu at (220.0, 92.5)
- added D27: WS2813, LED_SMD:LED_WS2812_PLCC6_5.0x5.0mm_P1.6mm, F.Cu at (220.0, 197.5)
- added D28: WS2813, LED_SMD:LED_WS2812_PLCC6_5.0x5.0mm_P1.6mm, F.Cu at (205.0, 107.5)
- added D29: WS2813, LED_SMD:LED_WS2812_PLCC6_5.0x5.0mm_P1.6mm, F.Cu at (205.0, 182.5)
- added D3: LED_Small, LED_SMD:LED_0603_1608Metric, F.Cu at (263.5, 211.8)
- added D30: WS2813, LED_SMD:LED_WS2812_PLCC6_5.0x5.0mm_P1.6mm, F.Cu at (265.0, 107.5)
- added D31: WS2813, LED_SMD:LED_WS2812_PLCC6_5.0x5.0mm_P1.6mm, F.Cu at (265.0, 182.5)
- added D32: WS2813, LED_SMD:LED_WS2812_PLCC6_5.0x5.0mm_P1.6mm, F.Cu at (190.0, 107.5)
- added D33: WS2813, LED_SMD:LED_WS2812_PLCC6_5.0x5.0mm_P1.6mm, F.Cu at (190.0, 182.5)
- added D34: WS2813, LED_SMD:LED_WS2812_PLCC6_5.0x5.0mm_P1.6mm, F.Cu at (250.0, 107.5)
- added D35: WS2813, LED_SMD:LED_WS2812_PLCC6_5.0x5.0mm_P1.6mm, F.Cu at (250.0, 182.5)
- added D36: WS2813, LED_SMD:LED_WS2812_PLCC6_5.0x5.0mm_P1.6mm, F.Cu at (175.0, 107.5)
- added D37: WS2813, LED_SMD:LED_WS2812_PLCC6_5.0x5.0mm_P1.6mm, F.Cu at (175.0, 182.5)
- added D38: WS2813, LED_SMD:LED_WS2812_PLCC6_5.0x5.0mm_P1.6mm, F.Cu at (235.0, 107.5)
- added D39: WS2813, LED_SMD:LED_WS2812_PLCC6_5.0x5.0mm_P1.6mm, F.Cu at (235.0, 182.5)
- added D4: WS2813, LED_SMD:LED_WS2812_PLCC6_5.0x5.0mm_P1.6mm, F.Cu at (205.0, 62.5)
- added D40: D_Schottky, Diode_SMD:D_SMA, F.Cu at (146.7, 68.0)
- added D41: WS2813, LED_SMD:LED_WS2812_PLCC6_5.0x5.0mm_P1.6mm, F.Cu at (160.0, 107.5)
- added D42: WS2813, LED_SMD:LED_WS2812_PLCC6_5.0x5.0mm_P1.6mm, F.Cu at (160.0, 182.5)
- added D43: WS2813, LED_SMD:LED_WS2812_PLCC6_5.0x5.0mm_P1.6mm, F.Cu at (220.0, 107.5)
- added D44: WS2813, LED_SMD:LED_WS2812_PLCC6_5.0x5.0mm_P1.6mm, F.Cu at (220.0, 182.5)
- added D45: WS2813, LED_SMD:LED_WS2812_PLCC6_5.0x5.0mm_P1.6mm, F.Cu at (205.0, 122.5)
- added D46: WS2813, LED_SMD:LED_WS2812_PLCC6_5.0x5.0mm_P1.6mm, F.Cu at (205.0, 167.5)
- added D47: WS2813, LED_SMD:LED_WS2812_PLCC6_5.0x5.0mm_P1.6mm, F.Cu at (280.0, 122.5)
- added D48: WS2813, LED_SMD:LED_WS2812_PLCC6_5.0x5.0mm_P1.6mm, F.Cu at (280.0, 167.5)
- added D49: WS2813, LED_SMD:LED_WS2812_PLCC6_5.0x5.0mm_P1.6mm, F.Cu at (190.0, 122.5)
- added D5: WS2813, LED_SMD:LED_WS2812_PLCC6_5.0x5.0mm_P1.6mm, F.Cu at (205.0, 227.5)
- added D50: WS2813, LED_SMD:LED_WS2812_PLCC6_5.0x5.0mm_P1.6mm, F.Cu at (190.0, 167.5)
- added D51: WS2813, LED_SMD:LED_WS2812_PLCC6_5.0x5.0mm_P1.6mm, F.Cu at (265.0, 122.5)
- added D52: WS2813, LED_SMD:LED_WS2812_PLCC6_5.0x5.0mm_P1.6mm, F.Cu at (265.0, 167.5)
- added D53: D_Schottky, Diode_SMD:D_SMA, F.Cu at (126.2, 82.1)
- added D54: WS2813, LED_SMD:LED_WS2812_PLCC6_5.0x5.0mm_P1.6mm, F.Cu at (175.0, 122.5)
- added D55: WS2813, LED_SMD:LED_WS2812_PLCC6_5.0x5.0mm_P1.6mm, F.Cu at (175.0, 167.5)
- added D56: WS2813, LED_SMD:LED_WS2812_PLCC6_5.0x5.0mm_P1.6mm, F.Cu at (250.0, 122.5)
- added D57: WS2813, LED_SMD:LED_WS2812_PLCC6_5.0x5.0mm_P1.6mm, F.Cu at (250.0, 167.5)
- added D58: WS2813, LED_SMD:LED_WS2812_PLCC6_5.0x5.0mm_P1.6mm, F.Cu at (160.0, 122.5)
- added D59: WS2813, LED_SMD:LED_WS2812_PLCC6_5.0x5.0mm_P1.6mm, F.Cu at (160.0, 167.5)
- added D6: WS2813, LED_SMD:LED_WS2812_PLCC6_5.0x5.0mm_P1.6mm, F.Cu at (220.0, 62.5)
- added D60: WS2813, LED_SMD:LED_WS2812_PLCC6_5.0x5.0mm_P1.6mm, F.Cu at (235.0, 122.5)
- added D61: WS2813, LED_SMD:LED_WS2812_PLCC6_5.0x5.0mm_P1.6mm, F.Cu at (235.0, 167.5)
- added D62: WS2813, LED_SMD:LED_WS2812_PLCC6_5.0x5.0mm_P1.6mm, F.Cu at (145.0, 122.5)
- added D63: WS2813, LED_SMD:LED_WS2812_PLCC6_5.0x5.0mm_P1.6mm, F.Cu at (145.0, 167.5)
- added D64: WS2813, LED_SMD:LED_WS2812_PLCC6_5.0x5.0mm_P1.6mm, F.Cu at (220.0, 122.5)
- added D65: WS2813, LED_SMD:LED_WS2812_PLCC6_5.0x5.0mm_P1.6mm, F.Cu at (220.0, 167.5)
- added D66: WS2813, LED_SMD:LED_WS2812_PLCC6_5.0x5.0mm_P1.6mm, F.Cu at (205.0, 137.5)
- added D67: WS2813, LED_SMD:LED_WS2812_PLCC6_5.0x5.0mm_P1.6mm, F.Cu at (205.0, 152.5)
- added D68: WS2813, LED_SMD:LED_WS2812_PLCC6_5.0x5.0mm_P1.6mm, F.Cu at (295.0, 137.5)
- added D69: WS2813, LED_SMD:LED_WS2812_PLCC6_5.0x5.0mm_P1.6mm, F.Cu at (295.0, 152.5)
- added D7: WS2813, LED_SMD:LED_WS2812_PLCC6_5.0x5.0mm_P1.6mm, F.Cu at (220.0, 227.5)
- added D70: WS2813, LED_SMD:LED_WS2812_PLCC6_5.0x5.0mm_P1.6mm, F.Cu at (190.0, 137.5)
- added D71: WS2813, LED_SMD:LED_WS2812_PLCC6_5.0x5.0mm_P1.6mm, F.Cu at (190.0, 152.5)
- added D72: WS2813, LED_SMD:LED_WS2812_PLCC6_5.0x5.0mm_P1.6mm, F.Cu at (280.0, 137.5)
- added D73: WS2813, LED_SMD:LED_WS2812_PLCC6_5.0x5.0mm_P1.6mm, F.Cu at (280.0, 152.5)
- added D74: WS2813, LED_SMD:LED_WS2812_PLCC6_5.0x5.0mm_P1.6mm, F.Cu at (175.0, 137.5)
- added D75: WS2813, LED_SMD:LED_WS2812_PLCC6_5.0x5.0mm_P1.6mm, F.Cu at (175.0, 152.5)
- added D76: WS2813, LED_SMD:LED_WS2812_PLCC6_5.0x5.0mm_P1.6mm, F.Cu at (265.0, 137.5)
- added D77: WS2813, LED_SMD:LED_WS2812_PLCC6_5.0x5.0mm_P1.6mm, F.Cu at (265.0, 152.5)
- added D78: WS2813, LED_SMD:LED_WS2812_PLCC6_5.0x5.0mm_P1.6mm, F.Cu at (160.0, 137.5)
- added D79: WS2813, LED_SMD:LED_WS2812_PLCC6_5.0x5.0mm_P1.6mm, F.Cu at (160.0, 152.5)
- added D8: WS2813, LED_SMD:LED_WS2812_PLCC6_5.0x5.0mm_P1.6mm, F.Cu at (205.0, 77.5)
- added D80: WS2813, LED_SMD:LED_WS2812_PLCC6_5.0x5.0mm_P1.6mm, F.Cu at (250.0, 137.5)
- added D81: WS2813, LED_SMD:LED_WS2812_PLCC6_5.0x5.0mm_P1.6mm, F.Cu at (250.0, 152.5)
- added D82: WS2813, LED_SMD:LED_WS2812_PLCC6_5.0x5.0mm_P1.6mm, F.Cu at (145.0, 137.5)
- added D83: WS2813, LED_SMD:LED_WS2812_PLCC6_5.0x5.0mm_P1.6mm, F.Cu at (145.0, 152.5)
- added D84: WS2813, LED_SMD:LED_WS2812_PLCC6_5.0x5.0mm_P1.6mm, F.Cu at (235.0, 137.5)
- added D85: WS2813, LED_SMD:LED_WS2812_PLCC6_5.0x5.0mm_P1.6mm, F.Cu at (235.0, 152.5)
- added D86: WS2813, LED_SMD:LED_WS2812_PLCC6_5.0x5.0mm_P1.6mm, F.Cu at (130.0, 137.5)
- added D87: WS2813, LED_SMD:LED_WS2812_PLCC6_5.0x5.0mm_P1.6mm, F.Cu at (130.0, 152.5)
- added D88: WS2813, LED_SMD:LED_WS2812_PLCC6_5.0x5.0mm_P1.6mm, F.Cu at (220.0, 137.5)
- added D89: WS2813, LED_SMD:LED_WS2812_PLCC6_5.0x5.0mm_P1.6mm, F.Cu at (220.0, 152.5)
- added D9: WS2813, LED_SMD:LED_WS2812_PLCC6_5.0x5.0mm_P1.6mm, F.Cu at (205.0, 212.5)
- added D90: D_Schottky, Diode_SMD:D_SMA, F.Cu at (274.3, 60.1)
- added D91: D_Schottky, Diode_SMD:D_SMA, F.Cu at (291.5, 79.5)
- added J1: Barrel_Jack_MountingPin, Connector_BarrelJack:BarrelJack_CUI_PJ-102AH_Horizontal, F.Cu at (168.2, 61.9)
- added J2: RJ45, Connector_RJ:RJ45_Amphenol_54602-x08_Horizontal, F.Cu at (290.0, 227.8)
- added J3: Conn_02x05_Odd_Even, Connector_PinHeader_2.54mm:PinHeader_2x05_P2.54mm_Vertical, F.Cu at (308.0, 193.0)
- added J4: Conn_02x04_Odd_Even, Connector_PinHeader_2.54mm:PinHeader_2x04_P2.54mm_Vertical, F.Cu at (298.5, 179.5)
- added J5: Conn_01x04_Male, Connector_JST:JST_PH_B4B-PH-K_1x04_P2.00mm_Vertical, F.Cu at (348.2, 150.5)
- added J6: Conn_01x04_Male, Connector_JST:JST_PH_B4B-PH-K_1x04_P2.00mm_Vertical, F.Cu at (348.2, 133.5)
- added J7: Conn_01x04_Male, Connector_JST:JST_PH_B4B-PH-K_1x04_P2.00mm_Vertical, F.Cu at (76.2, 156.2)
- added J8: Conn_01x04_Male, Connector_JST:JST_PH_B4B-PH-K_1x04_P2.00mm_Vertical, F.Cu at (76.2, 139.8)
- added L1: SDFL2012Q1R0KTF, Inductor_SMD:L_0805_2012Metric, F.Cu at (280.4, 234.6)
- added L2: 33u, Inductor_SMD:L_12x12mm_H8mm, F.Cu at (150.2, 56.0)
- added L3: 33u, Inductor_SMD:L_12x12mm_H8mm, F.Cu at (123.4, 93.6)
- added L4: 33u, Inductor_SMD:L_12x12mm_H8mm, F.Cu at (136.7, 56.0)
- added L5: 33u, Inductor_SMD:L_12x12mm_H8mm, F.Cu at (137.0, 93.6)
- added L6: 33u, Inductor_SMD:L_12x12mm_H8mm, F.Cu at (263.1, 56.1)
- added L7: 33u, Inductor_SMD:L_12x12mm_H8mm, F.Cu at (263.0, 69.9)
- added L8: 33u, Inductor_SMD:L_12x12mm_H8mm, F.Cu at (302.8, 84.4)
- added L9: 33u, Inductor_SMD:L_12x12mm_H8mm, F.Cu at (302.8, 70.8)
- added R1: 0R, Resistor_SMD:R_0603_1608Metric, F.Cu at (310.5, 95.0)
- added R10: 330R, Resistor_SMD:R_0603_1608Metric, F.Cu at (343.2, 157.8)
- added R11: 330R, Resistor_SMD:R_0603_1608Metric, F.Cu at (343.2, 138.0)
- added R12: 330R, Resistor_SMD:R_0603_1608Metric, F.Cu at (343.2, 141.0)
- added R13: 100R, Resistor_SMD:R_0603_1608Metric, F.Cu at (336.8, 158.5)
- added R14: 100R, Resistor_SMD:R_0603_1608Metric, F.Cu at (336.2, 142.0)
- added R15: 33k, Resistor_SMD:R_0603_1608Metric, F.Cu at (336.8, 150.5)
- added R16: 10k, Resistor_SMD:R_0603_1608Metric, F.Cu at (336.8, 148.8)
- added R17: 33k, Resistor_SMD:R_0603_1608Metric, F.Cu at (336.2, 134.0)
- added R18: 10k, Resistor_SMD:R_0603_1608Metric, F.Cu at (336.2, 132.0)
- added R19: 470R, Resistor_SMD:R_0603_1608Metric, F.Cu at (81.8, 157.8)
- added R2: 10k, Resistor_SMD:R_0603_1608Metric, F.Cu at (303.0, 166.2)
- added R20: 470R, Resistor_SMD:R_0603_1608Metric, F.Cu at (81.2, 141.0)
- added R21: 330R, Resistor_SMD:R_0603_1608Metric, F.Cu at (81.8, 151.8)
- added R22: 330R, Resistor_SMD:R_0603_1608Metric, F.Cu at (81.8, 148.8)
- added R23: 330R, Resistor_SMD:R_0603_1608Metric, F.Cu at (81.2, 135.2)
- added R24: 330R, Resistor_SMD:R_0603_1608Metric, F.Cu at (81.2, 132.2)
- added R25: 100R, Resistor_SMD:R_0603_1608Metric, F.Cu at (88.8, 147.2)
- added R26: 100R, Resistor_SMD:R_0603_1608Metric, F.Cu at (87.8, 131.3)
- added R27: 33k, Resistor_SMD:R_0603_1608Metric, F.Cu at (88.8, 155.2)
- added R28: 10k, Resistor_SMD:R_0603_1608Metric, F.Cu at (88.8, 157.2)
- added R29: 33k, Resistor_SMD:R_0603_1608Metric, F.Cu at (88.0, 139.2)
- added R3: 220R, Resistor_SMD:R_0603_1608Metric, F.Cu at (277.5, 196.0)
- added R30: 10k, Resistor_SMD:R_0603_1608Metric, F.Cu at (88.0, 141.2)
- added R31: 360R, Resistor_SMD:R_0603_1608Metric, F.Cu at (301.0, 219.8)
- added R32: 120R, Resistor_SMD:R_0603_1608Metric, F.Cu at (304.0, 219.8)
- added R33: 360R, Resistor_SMD:R_0603_1608Metric, F.Cu at (307.0, 219.8)
- added R34: 360R, Resistor_SMD:R_0603_1608Metric, F.Cu at (283.0, 219.8)
- added R35: 120R, Resistor_SMD:R_0603_1608Metric, F.Cu at (286.0, 219.8)
- added R36: 360R, Resistor_SMD:R_0603_1608Metric, F.Cu at (289.0, 219.8)
- added R37: 0R, Resistor_SMD:R_0603_1608Metric, F.Cu at (295.0, 209.5)
- added R38: 360R, Resistor_SMD:R_0603_1608Metric, F.Cu at (292.0, 219.8)
- added R39: 120R, Resistor_SMD:R_0603_1608Metric, F.Cu at (295.0, 219.8)
- added R4: 270R, Resistor_SMD:R_0603_1608Metric, F.Cu at (267.0, 205.8)
- added R40: 360R, Resistor_SMD:R_0603_1608Metric, F.Cu at (298.0, 219.8)
- added R41: 0R, Resistor_SMD:R_0603_1608Metric, F.Cu at (302.0, 209.5)
- added R42: 0R, Resistor_SMD:R_0603_1608Metric, F.Cu at (288.3, 209.8)
- added R5: 270R, Resistor_SMD:R_0603_1608Metric, F.Cu at (267.0, 208.8)
- added R6: 270R, Resistor_SMD:R_0603_1608Metric, F.Cu at (267.0, 211.8)
- added R7: 470R, Resistor_SMD:R_0603_1608Metric, F.Cu at (343.2, 148.5)
- added R8: 470R, Resistor_SMD:R_0603_1608Metric, F.Cu at (343.2, 132.0)
- added R9: 330R, Resistor_SMD:R_0603_1608Metric, F.Cu at (343.2, 154.8)
- added SW1: SW_Push, Button_Switch_THT:SW_PUSH-12mm, F.Cu at (319.2, 183.0)
- added SW2: SW_Push, Button_Switch_THT:SW_PUSH-12mm, F.Cu at (319.2, 168.5)
- added TP1: TestPoint, TestPoint:TestPoint_Pad_D2.5mm, F.Cu at (305.5, 231.0)
- added TP10: TestPoint, TestPoint:TestPoint_Pad_D2.5mm, F.Cu at (326.5, 136.0)
- added TP11: TestPoint, TestPoint:TestPoint_Pad_D2.5mm, F.Cu at (326.5, 152.5)
- added TP12: TestPoint, TestPoint:TestPoint_Pad_D2.5mm, F.Cu at (99.5, 132.0)
- added TP13: TestPoint, TestPoint:TestPoint_Pad_D2.5mm, F.Cu at (99.5, 149.0)
- added TP14: TestPoint, TestPoint:TestPoint_Pad_D2.5mm, F.Cu at (313.0, 222.0)
- added TP2: TestPoint, TestPoint:TestPoint_Pad_D2.5mm, F.Cu at (159.0, 55.0)
- added TP3: TestPoint, TestPoint:TestPoint_Pad_D2.5mm, F.Cu at (176.5, 55.0)
- added TP4: TestPoint, TestPoint:TestPoint_Pad_D2.5mm, F.Cu at (276.5, 224.5)
- added TP5: TestPoint, TestPoint:TestPoint_Pad_D2.5mm, F.Cu at (272.0, 236.5)
- added TP6: TestPoint, TestPoint:TestPoint_Pad_D2.5mm, F.Cu at (196.0, 62.5)
- added TP7: TestPoint, TestPoint:TestPoint_Pad_D2.5mm, F.Cu at (196.5, 227.5)
- added TP8: TestPoint, TestPoint:TestPoint_Pad_D2.5mm, F.Cu at (230.0, 62.5)
- added TP9: TestPoint, TestPoint:TestPoint_Pad_D2.5mm, F.Cu at (230.0, 227.5)
- added U1: 74HCT245, Package_SO:SOIC-20W_7.5x12.8mm_P1.27mm, F.Cu at (294.5, 191.0)
- added U10: LMV321, Package_TO_SOT_SMD:SOT-23-5, F.Cu at (333.0, 149.5)
- added U11: LMV321, Package_TO_SOT_SMD:SOT-23-5, F.Cu at (332.8, 133.0)
- added U12: INA826, Package_SO:SOIC-8_3.9x4.9mm_P1.27mm, F.Cu at (90.8, 151.2)
- added U13: INA826, Package_SO:SOIC-8_3.9x4.9mm_P1.27mm, F.Cu at (90.0, 135.2)
- added U14: LMV321, Package_TO_SOT_SMD:SOT-23-5, F.Cu at (92.2, 156.2)
- added U15: LMV321, Package_TO_SOT_SMD:SOT-23-5, F.Cu at (91.8, 140.2)
- added U16: XL1509-5.0E1, Package_SO:SOIC-8_3.9x4.9mm_P1.27mm, F.Cu at (121.2, 82.1)
- added U17: XL1509-5.0E1, Package_SO:SOIC-8_3.9x4.9mm_P1.27mm, F.Cu at (274.3, 55.3)
- added U18: XL1509-5.0E1, Package_SO:SOIC-8_3.9x4.9mm_P1.27mm, F.Cu at (291.4, 85.2)
- added U2: STM32F303K6Tx, Package_QFP:LQFP-32_7x7mm_P0.8mm, F.Cu at (277.2, 202.2)
- added U3: AMS1117-3.3, Package_TO_SOT_SMD:SOT-223-3_TabPin2, F.Cu at (282.3, 227.8)
- added U4: SP3485EN, Package_SO:SOIC-8_3.9x4.9mm_P1.27mm, F.Cu at (302.0, 214.2)
- added U5: SP3485EN, Package_SO:SOIC-8_3.9x4.9mm_P1.27mm, F.Cu at (288.0, 214.2)
- added U6: SP3485EN, Package_SO:SOIC-8_3.9x4.9mm_P1.27mm, F.Cu at (295.0, 214.2)
- added U7: XL1509-5.0E1, Package_SO:SOIC-8_3.9x4.9mm_P1.27mm, F.Cu at (151.7, 68.0)
- added U8: INA826, Package_SO:SOIC-8_3.9x4.9mm_P1.27mm, F.Cu at (334.5, 154.5)
- added U9: INA826, Package_SO:SOIC-8_3.9x4.9mm_P1.27mm, F.Cu at (334.2, 138.0)
- added Y1: 8MHz, Crystal:Crystal_SMD_5032-2Pin_5.0x3.2mm, F.Cu at (278.5, 193.2)
Routing:
- net GND: track 0.00 -> 267.7 mm, vias 0 -> 259
- net SENS4: track 0.00 -> 248.6 mm, vias 0 -> 2
- net GNDA: track 0.00 -> 247.3 mm, vias 0 -> 25
- net SENS3: track 0.00 -> 237.1 mm, vias 0 -> 2
- net LEDA: track 0.00 -> 190.3 mm, vias 0 -> 2
- net +3.3VA: track 0.00 -> 173.1 mm, vias 0 -> 9
- net LEDC: track 0.00 -> 168.6 mm, vias 0 -> 2
- net LEDB: track 0.00 -> 116.1 mm, vias 0 -> 2
- net Net-(D65-Pad3): track 0.00 -> 112.8 mm
- net +5V: track 0.00 -> 107.4 mm, vias 0 -> 2
- net Net-(D61-Pad3): track 0.00 -> 107.4 mm
- net Net-(D44-Pad3): track 0.00 -> 104.1 mm
- net LEDD: track 0.00 -> 99.3 mm, vias 0 -> 2
- net SENS2: track 0.00 -> 99.2 mm, vias 0 -> 2
- net Net-(D39-Pad3): track 0.00 -> 94.8 mm
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- added copper zone on B.Cu, net +24V
- added copper zone on F.Cu, net +24V
- added copper zone on In2.Cu, net +3.3VA
- added copper zone on In2.Cu, net +3V3
- added copper zone on F.Cu, net 5VD_1
- added copper zone on In2.Cu, net 5VD_1
- added copper zone on F.Cu, net 5VD_2
- added copper zone on In2.Cu, net 5VD_2
- added copper zone on F.Cu, net 5VD_3
- added copper zone on In2.Cu, net 5VD_3
- added copper zone on F.Cu, net 5VD_4
- added copper zone on In2.Cu, net 5VD_4
- added copper zone on F.Cu, net GND
- added copper zone on In1.Cu, net GND
- added copper zone on In1.Cu, net GNDA
- added copper zone on F.Cu, net Net-(L2-Pad2)
- added copper zone on F.Cu, net Net-(L3-Pad2)
- added copper zone on F.Cu, net Net-(L6-Pad2)
- added copper zone on F.Cu, net Net-(L8-Pad2)
Other:
- board outline added: 281 x 195 mm
- copper layers 2 -> 4
- board text added: "24V"
- board text added: "3.3V"
- board text added: "3.3VA"
- board text added: "5V"
- board text added: "5V Outputs"
- board text added: "5VD_1"
- board text added: "5VD_2"
- board text added: "5VD_3"
- board text added: "5VD_4"
- board text added: "Boot"
- board text added: "Debug"
- board text added: "GND"
- board text added: "GNDA"
- board text added: "GNDS"
- board text added: "RE:Flex Dance Panel Board v0.2, Designed by Brittany, Sept. 2020."
- board text added: "Reset"
- board text added: "Sensor DL"
- board text added: "Sensor DR"
- board text added: "Sensor UL"
- board text added: "Sensor UR"

Commit message: Transceiver fix + output mask
Connections:
- U4 pad 2: RX_EN -> GNDA
- U5 pad 2: TX_EN -> GNDA
- U6 pad 2: CK_EN -> GNDA
Routing:
- net GNDA: track 247.3 -> 256.7 mm, vias 25 -> 28
- net RX_EN: track 32.1 -> 30.9 mm
- net CK_EN: track 20.1 -> 18.8 mm
- net TX_EN: track 16.7 -> 15.9 mm
Changed lines of the file:
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@@
     (thickness 1.6)
     (drawings 138)
-    (tracks 2962)
+    (tracks 2976)
     (zones 0)
     (modules 323)
@@
   (page A3)
   (layers
-    (0 F.Cu signal hide)
-    (1 In1.Cu power hide)
+    (0 F.Cu signal)
+    (1 In1.Cu power)
     (2 In2.Cu power)
-    (31 B.Cu signal hide)
-    (33 F.Adhes user)
+    (31 B.Cu signal)
+    (33 F.Adhes user hide)
     (35 F.Paste user)
     (37 F.SilkS user)
     (39 F.Mask user)
-    (40 Dwgs.User user)
-    (41 Cmts.User user)
-    (42 Eco1.User user)
-    (43 Eco2.User user)
+    (40 Dwgs.User user hide)
+    (41 Cmts.User user hide)
+    (42 Eco1.User user hide)
+    (43 Eco2.User user hide)
     (44 Edge.Cuts user)
-    (45 Margin user)
-    (46 B.CrtYd user)
-    (47 F.CrtYd user)
+    (45 Margin user hide)
+    (46 B.CrtYd user hide)
+    (47 F.CrtYd user hide)
     (49 F.Fab user hide)
   )
@@
     (visible_elements 7FFFFFFF)
     (pcbplotparams
-      (layerselection 0x010fc_ffffffff)
+      (layerselection 0x010a8_ffffffff)
       (usegerberextensions false)
       (usegerberattributes false)
@@
       (outputformat 1)
       (mirror false)
-      (drillshape 1)
+      (drillshape 0)
       (scaleselection 1)
-      (outputdirectory ""))
+      (outputdirectory "gerber/"))
   )
   (net 0 "")
@@
       (net 266 RX_EN))
     (pad 2 smd roundrect (at -2.475 -0.635 270) (size 1.95 0.6) (layers F.Cu F.Paste F.Mask) (roundrect_rratio 0.25)
-      (net 266 RX_EN))
+      (net 1 GNDA))
     (pad 1 smd roundrect (at -2.475 -1.905 270) (size 1.95 0.6) (layers F.Cu F.Paste F.Mask) (roundrect_rratio 0.25)
       (net 249 UART_RX))
@@
       (net 265 TX_EN))
     (pad 2 smd roundrect (at -2.475 -0.635 270) (size 1.95 0.6) (layers F.Cu F.Paste F.Mask) (roundrect_rratio 0.25)
-      (net 265 TX_EN))
+      (net 1 GNDA))
     (pad 1 smd roundrect (at -2.475 -1.905 270) (size 1.95 0.6) (layers F.Cu F.Paste F.Mask) (roundrect_rratio 0.25)
       (net 251 "Net-(R42-Pad1)"))
@@
       (net 248 "Net-(R37-Pad1)"))
     (pad 2 smd roundrect (at -2.475 -0.635 270) (size 1.95 0.6) (layers F.Cu F.Paste F.Mask) (roundrect_rratio 0.25)
-      (net 267 CK_EN))
+      (net 1 GNDA))
     (pad 3 smd roundrect (at -2.475 0.635 270) (size 1.95 0.6) (layers F.Cu F.Paste F.Mask) (roundrect_rratio 0.25)
       (net 267 CK_EN))
@@
   (segment (start 334.2875 158.5) (end 335.7875 160) (width 0.25) (layer F.Cu) (net 1))
   (segment (start 335.7875 160) (end 338.25 160) (width 0.25) (layer F.Cu) (net 1))
+  (via (at 289.875 213.599694) (size 0.8) (drill 0.4) (layers F.Cu B.Cu) (net 1))
+  (segment (start 288.635 211.775) (end 288.635 212.359694) (width 0.25) (layer F.Cu) (net 1))
+  (segment (start 288.635 212.359694) (end 289.875 213.599694) (width 0.25) (layer F.Cu) (net 1))
+  (via (at 298.011784 211.907597) (size 0.8) (drill 0.4) (layers F.Cu B.Cu) (net 1))
+  (segment (start 296.00571 212.14571) (end 296.00571 212.8093) (width 0.25) (layer F.Cu) (net 1))
+  (segment (start 295.635 211.775) (end 296.00571 212.14571) (width 0.25) (layer F.Cu) (net 1))
+  (segment (start 296.00571 212.8093) (end 296.27142 213.07501) (width 0.25) (layer F.Cu) (net 1))
+  (segment (start 296.27142 213.07501) (end 297.251758 213.07501) (width 0.25) (layer F.Cu) (net 1))
+  (segment (start 297.251758 213.07501) (end 298.011784 212.314984) (width 0.25) (layer F.Cu) (net 1))
+  (segment (start 298.011784 212.314984) (end 298.011784 211.907597) (width 0.25) (layer F.Cu) (net 1))
+  (via (at 304.75 213.5) (size 0.8) (drill 0.4) (layers F.Cu B.Cu) (net 1))
+  (segment (start 303.983232 213.5) (end 304.75 213.5) (width 0.25) (layer F.Cu) (net 1))
+  (segment (start 303.00571 212.522478) (end 303.983232 213.5) (width 0.25) (layer F.Cu) (net 1))
+  (segment (start 302.635 211.775) (end 303.00571 212.14571) (width 0.25) (layer F.Cu) (net 1))
+  (segment (start 303.00571 212.14571) (end 303.00571 212.522478) (width 0.25) (layer F.Cu) (net 1))
   (segment (start 264.2875 205.75) (end 266.2125 205.75) (width 0.25) (layer F.Cu) (net 2))
   (segment (start 264.2875 208.75) (end 266.2125 208.75) (width 0.25) (layer F.Cu) (net 3))
@@
   (segment (start 299.095 186.5) (end 299.15 186.555) (width 0.25) (layer F.Cu) (net 264))
   (segment (start 297 186.5) (end 299.095 186.5) (width 0.25) (layer F.Cu) (net 264))
-  (segment (start 287.365 211.775) (end 288.635 211.775) (width 0.25) (layer F.Cu) (net 265))
   (via (at 285.75 209.25) (size 0.8) (drill 0.4) (layers F.Cu B.Cu) (net 265))
-  (segment (start 285.75 209.25) (end 279.47501 209.25) (width 0.25) (layer B.Cu) (net 265))
+  (via (at 277.75 207.52499) (size 0.8) (drill 0.4) (layers F.Cu B.Cu) (net 265))
   (segment (start 277.65 206.425) (end 277.65 207.42499) (width 0.25) (layer F.Cu) (net 265))
   (segment (start 277.65 207.42499) (end 277.75 207.52499) (width 0.25) (layer F.Cu) (net 265))
-  (segment (start 278.149999 207.924989) (end 277.75 207.52499) (width 0.25) (layer B.Cu) (net 265))
-  (via (at 277.75 207.52499) (size 0.8) (drill 0.4) (layers F.Cu B.Cu) (net 265))
   (segment (start 279.47501 209.25) (end 278.149999 207.924989) (width 0.25) (layer B.Cu) (net 265))
-  (segment (start 288.635 210.553994) (end 288.635 211.775) (width 0.25) (layer F.Cu) (net 265))
-  (segment (start 288.26251 210.181504) (end 288.635 210.553994) (width 0.25) (layer F.Cu) (net 265))
-  (segment (start 288.26251 209.218536) (end 288.26251 210.181504) (width 0.25) (layer F.Cu) (net 265))
+  (segment (start 285.75 209.25) (end 279.47501 209.25) (width 0.25) (layer B.Cu) (net 265))
+  (segment (start 278.149999 207.924989) (end 277.75 207.52499) (width 0.25) (layer B.Cu) (net 265))
+  (segment (start 287.365 210.635) (end 287.365 211.775) (width 0.25) (layer F.Cu) (net 265))
+  (segment (start 286.149999 208.850001) (end 287.893975 208.850001) (width 0.25) (layer F.Cu) (net 265))
   (segment (start 287.893975 208.850001) (end 288.26251 209.218536) (width 0.25) (layer F.Cu) (net 265))
   (segment (start 285.75 209.25) (end 286.149999 208.850001) (width 0.25) (layer F.Cu) (net 265))
-  (segment (start 286.149999 208.850001) (end 287.893975 208.850001) (width 0.25) (layer F.Cu) (net 265))
-  (segment (start 301.365 211.775) (end 302.635 211.775) (width 0.25) (layer F.Cu) (net 266))
+  (segment (start 288.26251 209.218536) (end 288.26251 210.231484) (width 0.25) (layer F.Cu) (net 265))
+  (segment (start 288.26251 210.231484) (end 287.943984 210.55001) (width 0.25) (layer F.Cu) (net 265))
+  (segment (start 287.44999 210.55001) (end 287.365 210.635) (width 0.25) (layer F.Cu) (net 265))
+  (segment (start 287.943984 210.55001) (end 287.44999 210.55001) (width 0.25) (layer F.Cu) (net 265))
   (segment (start 279.552198 207.950021) (end 280.547802 207.950021) (width 0.25) (layer F.Cu) (net 266))
   (segment (start 278.45 206.425) (end 278.45 207.275) (width 0.25) (layer F.Cu) (net 266))
@@
   (segment (start 280.697834 207.799989) (end 287.200011 207.799989) (width 0.25) (layer F.Cu) (net 266))
   (segment (start 290 205) (end 298.5 205) (width 0.25) (layer F.Cu) (net 266))
-  (segment (start 294.365 211.775) (end 295.635 211.775) (width 0.25) (layer F.Cu) (net 267))
   (via (at 287.25 205.25) (size 0.8) (drill 0.4) (layers F.Cu B.Cu) (net 267))
   (segment (start 281.425 205.05) (end 287.05 205.05) (width 0.25) (layer F.Cu) (net 267))
