File: led-board/led-board.kicad_pcb (KiCad board)
At the start: 4 copper layers, 281 x 195 mm, 323 parts, among them J1 Barrel_Jack_MountingPin, J2 RJ45, J3 Conn_02x05_Odd_Even, J4 Conn_02x04_Odd_Even, J5 Conn_01x04_Male, J6 Conn_01x04_Male, J7 Conn_01x04_Male, J8 Conn_01x04_Male, SW1 SW_Push, SW2 SW_Push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

Commit message: Post v0.2 order commit
Parts:
- C11, C110, C111, C19, C73, C74: footprint Capacitor_SMD:C_0603_1608Metric -> Capacitor_SMD:C_0805_2012Metric
- L2, L3, L4, L5, L6, L7, L8, L9: value 33u -> 47u
- U2: value STM32F303K6Tx -> STM32F334K8Tx
- moved C11 0.25 mm to (284.5, 222.2)
- moved C19 0.25 mm to (280.5, 222.2)
- moved R18 0.25 mm to (336.5, 132.0)
- moved R27 0.25 mm to (88.5, 155.2)
- moved R28 0.25 mm to (88.5, 157.2)
Connections:
- U10 pad 2: +3.3VA -> GNDA
- U10 pad 5: GNDA -> +3.3VA
- U11 pad 2: +3.3VA -> GNDA
- U11 pad 5: GNDA -> +3.3VA
- U14 pad 2: +3.3VA -> GNDA
- U14 pad 5: GNDA -> +3.3VA
- U15 pad 2: +3.3VA -> GNDA
- U15 pad 5: GNDA -> +3.3VA
Routing:
- net +3.3VA: track 173.1 -> 170.7 mm
- net Net-(U10-Pad3): track 8.86 -> 9.86 mm
- net Net-(U11-Pad3): track 9.67 -> 10.7 mm
- net Net-(U12-Pad6): track 10.8 -> 9.86 mm
- net +3V3: track 85.0 -> 84.1 mm, vias 6 -> 5
- net GNDA: track 256.7 -> 255.9 mm
