File: pcb/led-board.kicad_pcb (KiCad board)
At the start: 4 copper layers, 281 x 195 mm, 323 parts, among them J1 Barrel_Jack_MountingPin, J2 RJ45, J3 Conn_02x05_Odd_Even, J4 Conn_02x04_Odd_Even, J5 Conn_01x04_Male, J6 Conn_01x04_Male, J7 Conn_01x04_Male, J8 Conn_01x04_Male, SW1 SW_Push, SW2 SW_Push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

Commit message: LEDs and ADC working, separately
Parts:
- J1: footprint Connector_BarrelJack:BarrelJack_CUI_PJ-102AH_Horizontal -> Connector_BarrelJack:BarrelJack_Wuerth_6941xx301002
- SW1, SW2: footprint Button_Switch_THT:SW_PUSH-12mm -> Button_Switch_THT:SW_PUSH_6mm
Connections:
- U6 pad 1: Net-(R37-Pad1) -> UART_CK
- U6 pad 4: UART_CK -> Net-(R37-Pad1)
Routing:
- net UART_CK: track 23.9 -> 33.1 mm, vias 0 -> 2
- net Net-(R37-Pad1): track 2.74 -> 11.7 mm, vias 0 -> 2
- net GNDA: track 255.9 -> 261.9 mm
- net NRST: track 83.4 -> 82.3 mm
