File: panel-board.kicad_pcb (KiCad board)
At the start: 4 copper layers, 281 x 195 mm, 323 parts, among them J1 Barrel_Jack_MountingPin, J2 RJ45, J3 Conn_02x05_Odd_Even, J4 Conn_02x04_Odd_Even, J5 Conn_01x04_Male, J6 Conn_01x04_Male, J7 Conn_01x04_Male, J8 Conn_01x04_Male, SW1 SW_Push, SW2 SW_Push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

Commit message: Supply power externally, and move sensor position
Parts:
- removed TP1: TestPoint, TestPoint:TestPoint_Pad_D2.5mm
- moved J3 80.7 mm to (240.4, 237.0)
- moved SW2 77.4 mm to (264.5, 223.2)
- moved SW1 73.8 mm to (264.5, 232.5)
- moved C2 70.5 mm to (261.2, 237.5), turned to 180 degrees
- moved R2 66.7 mm to (258.0, 215.5), turned to 90 degrees
- moved J8 47.1 mm to (119.8, 121.8), turned to 270 degrees
- moved J5 46.5 mm to (305.2, 168.2), turned to 90 degrees
- moved J7 43.9 mm to (119.8, 162.2), turned to 270 degrees
- moved J6 43.4 mm to (305.2, 127.8), turned to 90 degrees
- moved R7 39.5 mm to (310.2, 170.2), turned to 0 degrees
- moved R20 39.3 mm to (114.8, 120.5), turned to 180 degrees
- moved R12 39.0 mm to (310.2, 120.2), turned to 180 degrees
- moved R22 38.7 mm to (114.2, 169.8), turned to 0 degrees
- moved C91 36.7 mm to (114.8, 123.2), turned to 0 degrees
- moved C51 36.6 mm to (310.2, 167.2), turned to 180 degrees
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Connections:
- C1 pad 1: +5V -> 5VD_4
- C11 pad 1: +5V -> 5VD_4
- J2 pad 7: +5V -> Net-(J2-Pad7)
- U1 pad 1: +5V -> 5VD_4
- U1 pad 20: +5V -> 5VD_4
- U3 pad 3: +5V -> 5VD_4
Routing:
- net +3.3VA: track 170.7 -> 645.8 mm, vias 9 -> 5
- net 5VD_4: track 88.9 -> 262.0 mm, vias 50 -> 60
- net +5V: track 107.5 -> 0.00 mm, vias 2 -> 0
- net SENS4: track 248.6 -> 294.5 mm
- net Net-(R2-Pad1): track 75.5 -> 36.6 mm
- net SWCLK: track 38.3 -> 60.8 mm, vias 0 -> 2
- net +3V3: track 84.1 -> 99.5 mm
- net SWDIO: track 42.5 -> 55.0 mm, vias 0 -> 4
- net GNDA: track 261.9 -> 270.1 mm, vias 28 -> 27
- net SENS1: track 86.0 -> 78.0 mm, vias 2 -> 0
- net NRST: track 82.3 -> 74.4 mm
- net SENS3: track 237.1 -> 242.8 mm
- net SENS2: track 99.2 -> 103.1 mm, vias 2 -> 0
- net UART_TX: track 19.8 -> 20.9 mm
- net Net-(R6-Pad1): track 18.4 -> 19.5 mm
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Other:
- outline, holes or cut-outs redrawn
