File: panel-board.kicad_pcb (KiCad board)
At the start: 4 copper layers, 281 x 195 mm, 318 parts, among them J1 Barrel_Jack_MountingPin, J2 RJ45, J3 Conn_02x05_Odd_Even, J4 Conn_02x04_Odd_Even, J5 Conn_01x04_Male, J6 Conn_01x04_Male, J7 Conn_01x04_Male, J8 Conn_01x04_Male, SW1 SW_Push, SW2 SW_Push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

Commit message: RS-485 transceiver fixes - production
Connections:
- net +3V3 renamed +3.3V
- D10 pad 1: Net-(D10-Pad1) -> unconnected-(D10-Pad1)
- D11 pad 1: Net-(D11-Pad1) -> unconnected-(D11-Pad1)
- D12 pad 1: Net-(D12-Pad1) -> unconnected-(D12-Pad1)
- D13 pad 1: Net-(D13-Pad1) -> unconnected-(D13-Pad1)
- D14 pad 1: Net-(D14-Pad1) -> unconnected-(D14-Pad1)
- D15 pad 1: Net-(D15-Pad1) -> unconnected-(D15-Pad1)
- D16 pad 1: Net-(D16-Pad1) -> unconnected-(D16-Pad1)
- D17 pad 1: Net-(D17-Pad1) -> unconnected-(D17-Pad1)
- D18 pad 1: Net-(D18-Pad1) -> unconnected-(D18-Pad1)
- D19 pad 1: Net-(D19-Pad1) -> unconnected-(D19-Pad1)
- D20 pad 1: Net-(D20-Pad1) -> unconnected-(D20-Pad1)
- D21 pad 1: Net-(D21-Pad1) -> unconnected-(D21-Pad1)
- D22 pad 1: Net-(D22-Pad1) -> unconnected-(D22-Pad1)
- D23 pad 1: Net-(D23-Pad1) -> unconnected-(D23-Pad1)
- D24 pad 1: Net-(D24-Pad1) -> unconnected-(D24-Pad1)
- D25 pad 1: Net-(D25-Pad1) -> unconnected-(D25-Pad1)
- D26 pad 1: Net-(D26-Pad1) -> unconnected-(D26-Pad1)
- D27 pad 1: Net-(D27-Pad1) -> unconnected-(D27-Pad1)
- D28 pad 1: Net-(D28-Pad1) -> unconnected-(D28-Pad1)
- D29 pad 1: Net-(D29-Pad1) -> unconnected-(D29-Pad1)
- D30 pad 1: Net-(D30-Pad1) -> unconnected-(D30-Pad1)
- D31 pad 1: Net-(D31-Pad1) -> unconnected-(D31-Pad1)
- D32 pad 1: Net-(D32-Pad1) -> unconnected-(D32-Pad1)
- D33 pad 1: Net-(D33-Pad1) -> unconnected-(D33-Pad1)
- D34 pad 1: Net-(D34-Pad1) -> unconnected-(D34-Pad1)
- D35 pad 1: Net-(D35-Pad1) -> unconnected-(D35-Pad1)
- D36 pad 1: Net-(D36-Pad1) -> unconnected-(D36-Pad1)
- D37 pad 1: Net-(D37-Pad1) -> unconnected-(D37-Pad1)
- D38 pad 1: Net-(D38-Pad1) -> unconnected-(D38-Pad1)
- D39 pad 1: Net-(D39-Pad1) -> unconnected-(D39-Pad1)
- D4 pad 1: Net-(D4-Pad1) -> unconnected-(D4-Pad1)
- D41 pad 1: Net-(D41-Pad1) -> unconnected-(D41-Pad1)
- D42 pad 1: Net-(D42-Pad1) -> unconnected-(D42-Pad1)
- D43 pad 1: Net-(D43-Pad1) -> unconnected-(D43-Pad1)
- D44 pad 1: Net-(D44-Pad1) -> unconnected-(D44-Pad1)
- D45 pad 1: Net-(D45-Pad1) -> unconnected-(D45-Pad1)
- D46 pad 1: Net-(D46-Pad1) -> unconnected-(D46-Pad1)
- D47 pad 1: Net-(D47-Pad1) -> unconnected-(D47-Pad1)
- D48 pad 1: Net-(D48-Pad1) -> unconnected-(D48-Pad1)
- D49 pad 1: Net-(D49-Pad1) -> unconnected-(D49-Pad1)
- D5 pad 1: Net-(D5-Pad1) -> unconnected-(D5-Pad1)
- D50 pad 1: Net-(D50-Pad1) -> unconnected-(D50-Pad1)
- D51 pad 1: Net-(D51-Pad1) -> unconnected-(D51-Pad1)
- D52 pad 1: Net-(D52-Pad1) -> unconnected-(D52-Pad1)
- D54 pad 1: Net-(D54-Pad1) -> unconnected-(D54-Pad1)
- D55 pad 1: Net-(D55-Pad1) -> unconnected-(D55-Pad1)
- D56 pad 1: Net-(D56-Pad1) -> unconnected-(D56-Pad1)
- D57 pad 1: Net-(D57-Pad1) -> unconnected-(D57-Pad1)
- D58 pad 1: Net-(D58-Pad1) -> unconnected-(D58-Pad1)
- D59 pad 1: Net-(D59-Pad1) -> unconnected-(D59-Pad1)
- D6 pad 1: Net-(D6-Pad1) -> unconnected-(D6-Pad1)
- D60 pad 1: Net-(D60-Pad1) -> unconnected-(D60-Pad1)
- D61 pad 1: Net-(D61-Pad1) -> unconnected-(D61-Pad1)
- D62 pad 1: Net-(D62-Pad1) -> unconnected-(D62-Pad1)
- D63 pad 1: Net-(D63-Pad1) -> unconnected-(D63-Pad1)
- D64 pad 1: Net-(D64-Pad1) -> unconnected-(D64-Pad1)
- D65 pad 1: Net-(D65-Pad1) -> unconnected-(D65-Pad1)
- D66 pad 1: Net-(D66-Pad1) -> unconnected-(D66-Pad1)
- D67 pad 1: Net-(D67-Pad1) -> unconnected-(D67-Pad1)
- D68 pad 1: Net-(D68-Pad1) -> unconnected-(D68-Pad1)
- D69 pad 1: Net-(D69-Pad1) -> unconnected-(D69-Pad1)
- D7 pad 1: Net-(D7-Pad1) -> unconnected-(D7-Pad1)
- D70 pad 1: Net-(D70-Pad1) -> unconnected-(D70-Pad1)
- D71 pad 1: Net-(D71-Pad1) -> unconnected-(D71-Pad1)
- D72 pad 1: Net-(D72-Pad1) -> unconnected-(D72-Pad1)
- D73 pad 1: Net-(D73-Pad1) -> unconnected-(D73-Pad1)
- D74 pad 1: Net-(D74-Pad1) -> unconnected-(D74-Pad1)
- D75 pad 1: Net-(D75-Pad1) -> unconnected-(D75-Pad1)
- D76 pad 1: Net-(D76-Pad1) -> unconnected-(D76-Pad1)
- D77 pad 1: Net-(D77-Pad1) -> unconnected-(D77-Pad1)
- D78 pad 1: Net-(D78-Pad1) -> unconnected-(D78-Pad1)
- D79 pad 1: Net-(D79-Pad1) -> unconnected-(D79-Pad1)
- D8 pad 1: Net-(D8-Pad1) -> unconnected-(D8-Pad1)
- D80 pad 1: Net-(D80-Pad1) -> unconnected-(D80-Pad1)
- D81 pad 1: Net-(D81-Pad1) -> unconnected-(D81-Pad1)
- D82 pad 1: Net-(D82-Pad1) -> unconnected-(D82-Pad1)
- D83 pad 1: Net-(D83-Pad1) -> unconnected-(D83-Pad1)
- D84 pad 1: Net-(D84-Pad1) -> unconnected-(D84-Pad1)
- D85 pad 1: Net-(D85-Pad1) -> unconnected-(D85-Pad1)
- D86 pad 1: Net-(D86-Pad1) -> unconnected-(D86-Pad1)
- D86 pad 3: Net-(D86-Pad3) -> unconnected-(D86-Pad3)
- D87 pad 1: Net-(D87-Pad1) -> unconnected-(D87-Pad1)
- D87 pad 3: Net-(D87-Pad3) -> unconnected-(D87-Pad3)
- D88 pad 1: Net-(D88-Pad1) -> unconnected-(D88-Pad1)
- D88 pad 3: Net-(D88-Pad3) -> unconnected-(D88-Pad3)
- D89 pad 1: Net-(D89-Pad1) -> unconnected-(D89-Pad1)
- D89 pad 3: Net-(D89-Pad3) -> unconnected-(D89-Pad3)
- D9 pad 1: Net-(D9-Pad1) -> unconnected-(D9-Pad1)
- J2 pad 4: Net-(J2-Pad4) -> unconnected-(J2-Pad4)
- J2 pad 5: Net-(J2-Pad5) -> unconnected-(J2-Pad5)
- J2 pad 7: Net-(J2-Pad7) -> unconnected-(J2-Pad7)
- J3 pad 10: Net-(J3-Pad10) -> unconnected-(J3-Pad10)
- J3 pad 3: Net-(J3-Pad3) -> unconnected-(J3-Pad3)
- J3 pad 9: Net-(J3-Pad9) -> unconnected-(J3-Pad9)
- U2 pad 18: Net-(U2-Pad18) -> unconnected-(U2-Pad18)
- U2 pad 25: Net-(U2-Pad25) -> unconnected-(U2-Pad25)
Routing:
- net Net-(U2-Pad25): track 5.91 -> 0.00 mm, vias 1 -> 0
- net UART_TX: track 22.4 -> 20.7 mm
- net GNDA: track 259.0 -> 257.7 mm
- net Net-(D13-Pad6): track 38.5 -> 37.4 mm
- net +3.3V: track 67.5 -> 66.4 mm
- net Net-(D34-Pad3): track 30.7 -> 29.8 mm
- net Net-(D22-Pad3): track 55.2 -> 54.5 mm
- net RX-: track 10.6 -> 9.98 mm
- net Net-(D14-Pad3): track 48.8 -> 48.3 mm
Other:
- net class Default removed
